Commit message: More generic 2R sim.py

File: 2R/2r_mx106/robot.urdf (robot description, URDF)
Before this commit: robot onshape, 5 links, 4 joints
Links:
- link base_106: geometry collision mesh filename=base.stl; collision mesh filename=dc08_m01_dummy.stl
- link first_segment_106: geometry collision mesh filename=dc08_m01_dummy.stl; collision mesh filename=ecrou_2.5.stl
- link sw_segment_106: geometry collision mesh filename=ecrou_4.stl; collision mesh filename=ecrou_4.stl
