Commit message: Multi-params adaptation

File: 2R/2r_erob/robot.urdf (robot description, URDF)
Before this commit: robot onshape, 4 links, 3 joints
Links:
- link base: mass 2.1622242401867124428 -> 2.1622242401867128869; geometry collision mesh filename=package:///80i_v5.stl; collision mesh filename=package:///bati_erob80.stl
- link bras1: mass 1.6401618924870369209 -> 1.6401618924870366989; geometry collision mesh filename=package:///bras1.stl; visual mesh filename=package:///bras1.stl
- link segment2: mass 12.857047818015505669 -> 12.857047818015507445; geometry collision mesh filename=package:///80i_v5.stl; collision mesh filename=package:///bras2.stl
Joints:
- removed joint r1
- removed joint r2
- added joint R1: type revolute, parent base, child bras1, origin xyz=-4.3051519674790368049e-17 -0.070436072480308878352 0.061999999999999430567 rpy=1.570796326794896558 -1.5707963267948954478 0, axis 0 0 1, limit effort=1 velocity=20
- added joint R2: type revolute, parent bras1, child segment2, origin xyz=-0.25000000000000005551 -4.305149412567801521e-17 -1.3877787807814456755e-17 rpy=-3.141592653589793116 5.0387059551511362915e-28 1.5707963267949036634, axis 0 0 1, limit effort=1 velocity=20
- joint end_frame: origin xyz=-2.9837244171328454876e-15 0.24999999999997310485 0.029999999999995238809 rpy=-1.1131317589294916161e-14 -3.1469101278800327038e-14 -1.5707963267948970021 -> xyz=-2.9837244171328454876e-15 -0.24999999999997310485 -0.029999999999995238809 rpy=3.1415926535897820138 3.1469101278800327038e-14 1.5707963267948970021
