Commit message: isaac identification rig

File: bam/isaac_identification_rig/assets/identification_rig_0_150m_1kg/robot.urdf (robot description, URDF)
Before this commit: robot onshape, 2 links, 1 joints
Joints:
- joint sts3215: limit lower=-1.7453292519943295336 upper=1.7453292519943295336 effort=1 velocity=20 -> lower=-1.7453292519943295336 upper=1.7453292519943295336
